File: keypad.kicad_pcb (KiCad board)
At the start: 2 copper layers, 67 x 111.8 mm, 10 parts, among them SW1 SW_Push, SW2 SW_Push, SW3 SW_Push, SW4 SW_Push, SW5 SW_Push, SW6 SW_Push, SW7 SW_Push, SW8 SW_Push, SW9 SW_Push, U1 ESP32-S3-DevKitC-1

Commit message: v1
Other:
- board text added: "v1.0"
Changed lines of the file:
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@@
 		(layer "Edge.Cuts")
+	)
+	(gr_text "v1.0"
+		(at 165.73 137.84 0)
+		(layer "F.SilkS")
+		(effects
+			(font
+				(size 1.5 1.5)
+				(thickness 0.2)
+			)
+			(justify left bottom)
+		)
 	)
 	(gr_text "gavhu10/keypad"
